Commit message: Adding Tilt Node

File: Base-Navigation/raker_base_ws/src/raker_base_description/urdf/HDL-32E.urdf.xacro (robot description, xacro)
@@ -2,5 +2,5 @@
 <robot xmlns:xacro="http://www.ros.org/wiki/xacro" name="HDL-32E">
   <xacro:property name="M_PI" value="3.1415926535897931" />
-  <xacro:macro name="HDL-32E" params="*origin parent:=base_link name:=velodyne topic:=/velodyne_points organize_cloud:=false hz:=10 lasers:=32 samples:=2187 collision_range:=0.3 min_range:=0.9 max_range:=130.0 noise:=0.008 min_angle:=-${M_PI} max_angle:=${M_PI} gpu:=false">
+  <xacro:macro name="HDL-32E" params="*origin parent:=base_link name:=velodyne topic:=/velodyne_points organize_cloud:=false hz:=10 lasers:=32 samples:=2187 collision_range:=0.3 min_range:=0.9 max_range:=130.0 noise:=0.008 min_angle:=-1.570795 max_angle:=1.570795 gpu:=false">
     <joint name="${name}_base_mount_joint" type="fixed">
       <xacro:insert_block name="origin" />

File: Base-Navigation/raker_base_ws/src/raker_base_description/urdf/husky.urdf.xacro (robot description, xacro)
@@ -118,5 +118,5 @@
   <xacro:husky_decorate />
   <xacro:if value="$(arg laser_enabled)">
-  	<xacro:include filename="$(find velodyne_description)/urdf/HDL-32E.urdf.xacro"/>
+  	<xacro:include filename="$(find raker_base_description)/urdf/HDL-32E.urdf.xacro"/>
   	<xacro:HDL-32E parent="base_link" name="velodyne" topic="/velodyne_points" organize_cloud="false" hz="10" samples="220" gpu="false" lasers="16" max_range="30">
     	  <origin xyz="0 0 0.4" rpy="0 0 0" />

Commit message: Adding Gradient Assesser code as well as Launch files for the LIDAR to PCD pipeline

File: Base-Navigation/raker_base_ws/src/raker_base_description/urdf/HDL-32E.urdf.xacro (robot description, xacro)
@@ -2,5 +2,5 @@
 <robot xmlns:xacro="http://www.ros.org/wiki/xacro" name="HDL-32E">
   <xacro:property name="M_PI" value="3.1415926535897931" />
-  <xacro:macro name="HDL-32E" params="*origin parent:=base_link name:=velodyne topic:=/velodyne_points organize_cloud:=false hz:=10 lasers:=32 samples:=2187 collision_range:=0.3 min_range:=0.9 max_range:=130.0 noise:=0.008 min_angle:=-1.570795 max_angle:=1.570795 gpu:=false">
+  <xacro:macro name="HDL-32E" params="*origin parent:=base_link name:=velodyne topic:=/velodyne_points organize_cloud:=false hz:=10 lasers:=32 samples:=2187 collision_range:=0.3 min_range:=0.9 max_range:=130.0 noise:=0.008 min_angle:=-0.7853975 max_angle:=0.7853975 gpu:=false">
     <joint name="${name}_base_mount_joint" type="fixed">
       <xacro:insert_block name="origin" />

File: Base-Navigation/raker_base_ws/src/raker_base_description/urdf/husky.urdf.xacro (robot description, xacro)
@@ -119,5 +119,5 @@
   <xacro:if value="$(arg laser_enabled)">
   	<xacro:include filename="$(find raker_base_description)/urdf/HDL-32E.urdf.xacro"/>
-  	<xacro:HDL-32E parent="base_link" name="velodyne" topic="/velodyne_points" organize_cloud="false" hz="10" samples="220" gpu="false" lasers="16" max_range="30">
+  	<xacro:HDL-32E parent="base_link" name="velodyne" topic="/velodyne_points" organize_cloud="false" hz="10" samples="220" gpu="false" lasers="16" max_range="10">
     	  <origin xyz="0 0 0.4" rpy="0 0 0" />
   	</xacro:HDL-32E>
